File: Design_ files/The Sixth Eye KiCAD/The Sixth Eye KiCAD.sch (KiCad schematic (older format))
At the start: 19 parts, among them J1 Vibration out, J2 Battery conn, J3 US Sensor conn., Q1 BC547, U1 LTC3525ISC6-5, U2 ATmega328-AU, U3 ADXL343, Y1 8Mhz

Commit message: KiCAD Pcb completed for Sixth_Eye including Accelerometer
Parts:
- J2: footprint Connector_Phoenix_MC:PhoenixContact_MC_1,5_2-G-3.5_1x02_P3.50mm_Horizontal -> Connector_JST:JST_XH_S2B-XH-A-1_1x02_P2.50mm_Horizontal
Changed lines of the file:
@@
 F 0 "J2" H 8500 1600 50  0000 C CNN
 F 1 "Battery conn" H 8250 1900 50  0000 C CNN
-F 2 "Connector_Phoenix_MC:PhoenixContact_MC_1,5_2-G-3.5_1x02_P3.50mm_Horizontal" H 8350 1800 50  0001 C CNN
+F 2 "Connector_JST:JST_XH_S2B-XH-A-1_1x02_P2.50mm_Horizontal" H 8350 1800 50  0001 C CNN
 F 3 "~" H 8350 1800 50  0001 C CNN
 	1    8350 1800
